File: pcb/H-Bridge.sch (EAGLE design)
At the start: 49 parts, among them IC1 L293D, T1_PNP BC337, T2_NPN BC327, T3_PNP BC337, T4_NPN BC327

Commit message: Add files via upload
Parts:
- added BLIND-1, BLIND-2, BLIND-3, BLIND-4: (no value), pinhead:PINHD-1X2
- T1_PNP, T3_PNP: value BC337 -> BC237; device transistor:BC327-40-PNP-TO92-EBC -> transistor-neu-to92:-PNP-TO92-CBE
- T2_NPN, T4_NPN, T_NPN: value BC327 -> BC337
- renumbered CONTROL_PINS1 to CONTROL, ENABLE1 to ENABLE, GND_PINS to GND, MOTOR_PIN1 to M1, MOTOR_PIN2 to M2, MOTOR_PIN3 to M3, VCC1 to EXT_VCC, VCC_SUPPLY_PIN to VCC
Connections:
- net GND: no longer LED1.C, LED3.C
- net N$10: now also LED3.C; no longer LED3.A
- net N$5: now also LED1.C; no longer LED1.A
- net VCC: now also LED1.A, LED3.A
